File: prototype/Boards/Transmit US/Transmit US.kicad_pcb (KiCad board)
At the start: 2 copper layers, 24 x 29 mm, 18 parts, among them J1 Header, U1 SN74AHC1G04QDCKRQ1, U2 ICL3232IVZ

Commit message: Adjustments to new logo
Parts:
- removed Ref**: Val**, uFinder:logo
- added Logo1: ~, uFinder:uFollowLogo, B.Cu at (110.7, 86.7)
