File: prototype/Boards/Transmit US/Transmit US.kicad_sch (KiCad schematic)
At the start: 17 parts, among them J1 Header, U1 SN74AHC1G04QDCKRQ1, U2 ICL3232IVZ

Commit message: Adjustments to new logo
Parts:
- added Logo1: ~, uFinder:uFollowLogo, symbol uFinder:Logo
