File: prototype/Boards/Receive MCU/receive mcu prototype r1/receive mcu prototype r1.kicad_pcb (KiCad board)
At the start: 2 copper layers, 70.6 x 65.3 mm, 35 parts, among them J1 Conn_01x04_Socket, J11 Conn_01x04_Socket, J2 Conn_01x04_Socket, J3 Conn_01x02_Socket, J4 USB_B_Micro, J5 Conn_01x20_Pin, J6 Conn_01x20_Pin, J7 Conn_01x04_Socket, Q2 Q_NPN_BEC, Q3 Q_NPN_BEC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

Commit message: gerbers and few updates
Parts:
- added Logo1: ~, uFinder:uFollowLogo, F.Cu at (112.7, 89.9)
Other:
- board text added: "Prototype v0.1"
- board text removed: "Ufollow Prototype r1"
