File: prototype/Boards/Receive MCU/receive mcu prototype r1/receive mcu prototype r1.kicad_sch (KiCad schematic)
At the start: 14 parts, among them J1 Conn_01x04_Socket, J11 Conn_01x04_Socket, J2 Conn_01x04_Socket, J5 Conn_01x20_Pin, J6 Conn_01x20_Pin, J7 Conn_01x04_Socket, SW2 SW_Push, U1 ESP32-S3-WROOM-1-N4R2

Commit message: gerbers and few updates
Parts:
- added Logo1: ~, uFinder:uFollowLogo, symbol uFinder:Logo
Changed lines of the file:
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@@
+    )
+  )
+  (symbol (lib_id "uFinder:Logo") (at 33.02 86.36 0) (unit 1)
+    (in_bom no) (on_board yes) (dnp no) (fields_autoplaced)
+    (property "Reference" "Logo1" (at 35.56 86.995 0)
+      (effects (font (size 1.27 1.27)) (justify left))
+    )
+    (property "Value" "~" (at 33.02 86.36 0)
+      (effects (font (size 1.27 1.27)))
+    )
+    (property "Footprint" "uFinder:uFollowLogo" (at 33.02 86.36 0)
+      (effects (font (size 1.27 1.27)) hide)
+    )
+    (property "Datasheet" "" (at 33.02 86.36 0)
+      (effects (font (size 1.27 1.27)) hide)
+    )
+    (instances
+      (project "receive mcu prototype r1"
+        (path "/6ff1ab3f-c90b-4acb-b3d7-b045de372bcb"
+          (reference "Logo1") (unit 1)
+        )
+      )
     )
   )
