File: prototype/Boards/Receive US v2/Receive US v2.kicad_pcb (KiCad board)
At the start: 2 copper layers, 38 x 31.7 mm, 47 parts, among them J1 Conn_01x04_Socket, Q1 MMBT3904, Q3 MMBT3904, U1 LM324

Commit message: Recv V2 layout
Parts:
- Logo1: moved to B.Cu
- TP1, TP2, TP3, TP4, TP5, TP6, TP7, TP8: footprint TestPoint:TestPoint_THTPad_D1.5mm_Drill0.7mm -> uFinder:TestPoint_THTPad_D1.5mm_Drill0.7mm; moved to B.Cu
- moved TP6 53.3 mm to (62.5, 64.5), turned to 180 degrees
- moved TP7 52.7 mm to (68.5, 50.1), turned to 180 degrees
- moved TP5 46.3 mm to (69.5, 69.3), turned to 180 degrees
- moved TP1 45.5 mm to (64.1, 74.7), turned to 180 degrees
- moved TP8 38.5 mm to (80.7, 70.2), turned to 180 degrees
- moved TP2 33.7 mm to (80.5, 49.5), turned to 180 degrees
- moved TP3 26.2 mm to (86.5, 71.0), turned to 180 degrees
- moved R11 25.7 mm to (59.0, 65.4), turned to -90 degrees
- moved TP4 23.9 mm to (90.8, 57.1), turned to 180 degrees
- moved C6 19.4 mm to (69.8, 64.5), turned to 90 degrees
- moved Logo1 18.8 mm to (62.5, 68.5), turned to 180 degrees
- moved R6 11.2 mm to (77.2, 70.1)
- moved C7 10.3 mm to (82.3, 65.1), turned to -90 degrees
- moved C8 9.85 mm to (79.7, 63.2), turned to 90 degrees
- moved R15 9.83 mm to (75.5, 57.2), turned to 0 degrees
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- renumbered Q3 to Q2
Routing:
- net /DATA: track 0.00 -> 42.9 mm, vias 0 -> 1
- net Net-(U1B-+): track 0.00 -> 41.9 mm
- net Net-(Q1-C): track 0.00 -> 38.4 mm, vias 0 -> 2
- net Net-(U1C--): track 0.00 -> 24.3 mm
- net Net-(C2-Pad1): track 0.00 -> 20.1 mm, vias 0 -> 2
- net Net-(U1B--): track 0.00 -> 18.8 mm
- net GND: track 0.00 -> 18.0 mm, vias 0 -> 12
- net Net-(R2-Pad2): track 0.00 -> 17.3 mm
- net +3.3V: track 0.00 -> 16.5 mm, vias 0 -> 1
- net Net-(D1-A): track 0.00 -> 16.1 mm
- net Net-(C3-Pad2): track 0.00 -> 15.3 mm
- net Net-(U1A-+): track 0.00 -> 15.3 mm
- net Net-(Q2-B): track 0.00 -> 13.1 mm
- net Net-(R7-Pad2): track 0.00 -> 11.8 mm
- net Net-(LS1-Pad1): track 0.00 -> 10.2 mm
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- added copper zone on F.Cu, net +3.3V
- added copper zone on B.Cu, net GND
Other:
- board text added: "3.3V"
- board text added: "DATA"
- board text added: "GND"
- board text added: "SQL"

Commit message: Clean up pours
Parts:
- moved R11 8.65 mm to (61.5, 57.1), turned to 90 degrees
- moved TP6 3.81 mm to (58.8, 65.5)
- moved R18 2.91 mm to (74.8, 53.7)
- moved D1 2.79 mm to (72.5, 53.7)
- moved R10 1.75 mm to (65.3, 52.0)
- moved R12 1.52 mm to (59.0, 57.1)
- moved Q1 0.71 mm to (62.3, 68.8)
Routing:
- net Net-(Q1-C): track 38.4 -> 28.9 mm
- net /DATA: track 42.9 -> 36.6 mm, vias 1 -> 0
- net Net-(U1A-+): track 15.3 -> 18.5 mm, vias 0 -> 1
- net +3.3V: track 16.5 -> 18.3 mm
