File: prototype/Boards/Receive US v2/Receive US v2.kicad_pcb (KiCad board)
At the start: 2 copper layers, 38 x 31.7 mm, 47 parts, among them J1 Conn_01x04_Socket, Q1 MMBT3904, Q3 MMBT3904, U1 LM324

Commit message: routed
Parts:
- Logo1: moved to B.Cu
- moved TP7 62.1 mm to (57.7, 55.6)
- moved TP6 55.2 mm to (61.0, 60.3)
- moved TP5 54.6 mm to (61.0, 63.5)
- moved TP1 43.9 mm to (66.0, 76.2)
- moved TP8 35.5 mm to (84.5, 76.2)
- moved TP2 34.7 mm to (79.8, 48.9)
- moved TP3 24.9 mm to (87.6, 69.8)
- moved TP4 24.4 mm to (87.6, 67.3)
- moved C6 17.3 mm to (74.9, 57.1), turned to 0 degrees
- moved Logo1 11.7 mm to (74.9, 66.3), turned to 180 degrees
- moved R15 5.08 mm to (66.0, 64.8), turned to 0 degrees
- moved R16 5.08 mm to (66.0, 49.5)
- moved Q1 4.45 mm to (61.0, 66.7)
- moved C4 4.44 mm to (79.4, 69.8), turned to 180 degrees
- moved C9 2.54 mm to (74.9, 50.8), turned to -90 degrees
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Routing:
- net /DATA: track 0.00 -> 52.5 mm
- net +3.3V: track 0.00 -> 48.8 mm, vias 0 -> 2
- net Net-(Q1-C): track 0.00 -> 37.8 mm
- net Net-(U1B-+): track 0.00 -> 36.9 mm
- net Net-(D1-A): track 0.00 -> 30.7 mm
- net Net-(C3-Pad2): track 0.00 -> 22.6 mm
- net GND: track 0.00 -> 21.7 mm, vias 0 -> 12
- net Net-(U1C--): track 0.00 -> 20.5 mm
- net Net-(U1B--): track 0.00 -> 18.5 mm, vias 0 -> 2
- net Net-(U1D--): track 0.00 -> 18.1 mm
- net Net-(U1A-+): track 0.00 -> 16.6 mm
- net Net-(C2-Pad1): track 0.00 -> 14.2 mm, vias 0 -> 2
- net Net-(R7-Pad2): track 0.00 -> 13.8 mm, vias 0 -> 2
- net Net-(Q1-B): track 0.00 -> 11.8 mm
- net Net-(R2-Pad2): track 0.00 -> 9.85 mm
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- added copper zone on B.Cu, net GND
Other:
- board size 38 x 31.7 mm -> 38.1 x 31.7 mm
- board text added: "2IN"
- board text added: "3IN"
- board text added: "3V3"
- board text added: "4IN"
- board text added: "4OUT"
- board text added: "DATA"
- board text added: "GND"
- board text added: "REF"
- board text added: "SQL"
