File: prototype/Boards/Receive US v2 elliot/Receive US v2 elliot.kicad_sch (KiCad schematic)
At the start: 47 parts, among them J1 Conn_01x04_Socket, Q1 MMBT3904, Q3 MMBT3904, U1 LM324

Commit message: my board
Parts:
- R19: now not fitted; now left out of the parts list
Changed lines of the file:
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@@
   )
   (symbol (lib_id "Device:R") (at 30.48 58.42 180) (unit 1)
-    (in_bom yes) (on_board yes) (dnp no) (fields_autoplaced)
+    (in_bom no) (on_board yes) (dnp yes) (fields_autoplaced)
     (property "Reference" "R19" (at 33.02 57.785 0)
       (effects (font (size 1.27 1.27)) (justify right))
