File: prototype/Boards/Receive US v2 elliot/Receive US v2 elliot-panel.kicad_pcb (KiCad board)
At the start: 2 copper layers, 96.5 x 86.4 mm, 188 parts, among them J1 Conn_01x04_Socket, Q1 MMBT3904, Q3 MMBT3904, U1 LM324

Commit message: panelized
Parts:
- removed the C1 at (105.4, 44.5)
- removed the C1 at (105.4, 76.2)
- removed the C2 at (105.4, 54.6)
- removed the C2 at (105.4, 86.4)
- removed the C3 at (105.4, 88.9)
- removed the C3 at (105.4, 57.1)
- removed the C4 at (101.0, 59.7)
- removed the C4 at (101.0, 91.4)
- removed the C5 at (87.6, 57.1)
- removed the C5 at (87.6, 88.9)
- removed the C6 at (96.5, 78.7)
- removed the C6 at (96.5, 47.0)
- removed the C7 at (110.5, 47.0)
- removed the C7 at (110.5, 78.7)
- removed the C8 at (110.5, 81.3)
- removed the C8 at (110.5, 49.5)
- removed the C9 at (96.5, 40.6)
- removed the C9 at (96.5, 72.4)
- removed the D1 at (94.0, 40.6)
- removed the D1 at (94.0, 72.4)
- removed the H1 at (81.3, 40.6)
- removed the H1 at (81.3, 72.4)
- removed the H2 at (111.8, 40.6)
- removed the H2 at (111.8, 72.4)
- removed the H3 at (81.3, 64.8)
- removed the H3 at (81.3, 96.5)
- removed the H4 at (111.8, 96.5)
- removed the H4 at (111.8, 64.8)
- removed the J1 at (92.8, 96.0)
- removed the J1 at (92.8, 64.2)
- removed the LS1 at (96.6, 46.9)
- removed the LS1 at (96.6, 78.7)
- removed the Logo1 at (96.5, 87.9)
- removed the Logo1 at (96.5, 56.1)
- removed the Q1 at (82.5, 56.5)
- removed the Q1 at (82.5, 88.3)
- removed the Q3 at (82.5, 78.7)
- removed the Q3 at (82.5, 47.0)
- removed the R1 at (105.4, 73.7)
- removed the R1 at (105.4, 41.9)
- removed the R10 at (87.6, 44.5)
- removed the R10 at (87.6, 76.2)
- removed the R11 at (105.4, 62.2)
- removed the R11 at (105.4, 94.0)
- removed the R12 at (87.6, 73.7)
- removed the R12 at (87.6, 41.9)
- removed the R13 at (110.5, 86.4)
- removed the R13 at (110.5, 54.6)
- removed the R14 at (110.5, 83.8)
- removed the R14 at (110.5, 52.1)
- removed the R15 at (87.6, 86.4)
- removed the R15 at (87.6, 54.6)
- removed the R16 at (87.6, 39.4)
- removed the R16 at (87.6, 71.1)
- removed the R17 at (87.6, 62.2)
- removed the R17 at (87.6, 94.0)
- removed the R18 at (99.1, 72.4)
- removed the R18 at (99.1, 40.6)
- removed the R19 at (105.4, 39.4)
- removed the R19 at (105.4, 71.1)
- removed the R2 at (105.4, 81.3)
- removed the R2 at (105.4, 49.5)
- removed the R3 at (105.4, 47.0)
- removed the R3 at (105.4, 78.7)
- removed the R4 at (105.4, 83.8)
- removed the R4 at (105.4, 52.1)
- removed the R5 at (105.4, 91.4)
- removed the R5 at (105.4, 59.7)
- removed the R6 at (87.6, 59.7)
- removed the R6 at (87.6, 91.4)
- removed the R7 at (87.6, 52.1)
- removed the R7 at (87.6, 83.8)
- removed the R8 at (87.6, 49.5)
- removed the R8 at (87.6, 81.3)
- removed the R9 at (87.6, 78.7)
- removed the R9 at (87.6, 47.0)
- removed the TP1 at (87.6, 97.8)
- removed the TP1 at (87.6, 66.0)
- removed the TP2 at (101.3, 70.5)
- removed the TP2 at (101.3, 38.7)
- removed the TP3 at (109.2, 91.4)
- removed the TP3 at (109.2, 59.7)
- removed the TP4 at (109.2, 88.9)
- removed the TP4 at (109.2, 57.1)
- removed the TP5 at (82.5, 53.3)
- removed the TP5 at (82.5, 85.1)
- removed the TP6 at (82.5, 50.2)
- removed the TP6 at (82.5, 81.9)
- removed the TP7 at (79.2, 45.5)
- removed the TP7 at (79.2, 77.2)
- removed the TP8 at (106.0, 66.0)
- removed the TP8 at (106.0, 97.8)
- removed the U1 at (96.5, 53.3)
- removed the U1 at (96.5, 85.1)
- added C1: 10nF, Capacitor_SMD:C_0805_2012Metric, F.Cu at (103.8, 60.7)
- added C1: 10nF, Capacitor_SMD:C_0805_2012Metric, F.Cu at (103.8, 92.5)
- added C2: 1nF, Capacitor_SMD:C_0805_2012Metric, F.Cu at (107.4, 50.8)
- added C2: 1nF, Capacitor_SMD:C_0805_2012Metric, F.Cu at (107.4, 82.6)
- added C3: 1nF, Capacitor_SMD:C_0805_2012Metric, F.Cu at (112.9, 78.5)
- added C3: 1nF, Capacitor_SMD:C_0805_2012Metric, F.Cu at (112.9, 46.8)
- added C4: 68pF, Capacitor_SMD:C_0603_1608Metric, F.Cu at (110.9, 78.4)
- added C4: 68pF, Capacitor_SMD:C_0603_1608Metric, F.Cu at (110.9, 46.6)
- added C5: 10nF, Capacitor_SMD:C_0805_2012Metric, F.Cu at (96.6, 44.2)
- added C5: 10nF, Capacitor_SMD:C_0805_2012Metric, F.Cu at (96.6, 76.0)
- added C6: 1uF, Capacitor_SMD:C_0805_2012Metric, F.Cu at (90.6, 52.4)
- added C6: 1uF, Capacitor_SMD:C_0805_2012Metric, F.Cu at (90.6, 84.1)
- added C7: 1nF, Capacitor_SMD:C_0805_2012Metric, F.Cu at (102.2, 51.2)
- added C7: 1nF, Capacitor_SMD:C_0805_2012Metric, F.Cu at (102.2, 83.0)
- added C8: 1uF, Capacitor_SMD:C_0805_2012Metric, F.Cu at (102.2, 85.4)
- added C8: 1uF, Capacitor_SMD:C_0805_2012Metric, F.Cu at (102.2, 53.6)
- added C9: 1nF, Capacitor_SMD:C_0805_2012Metric, F.Cu at (90.6, 54.9)
- added C9: 1nF, Capacitor_SMD:C_0805_2012Metric, F.Cu at (90.6, 86.6)
- added D1: LED, LED_SMD:LED_0805_2012Metric, F.Cu at (92.4, 63.3)
- added D1: LED, LED_SMD:LED_0805_2012Metric, F.Cu at (92.4, 95.0)
- added H1: MountingHole, MountingHole:MountingHole_3.2mm_M3, F.Cu at (81.2, 40.6)
- added H1: MountingHole, MountingHole:MountingHole_3.2mm_M3, F.Cu at (81.2, 72.3)
- added H2: MountingHole, MountingHole:MountingHole_3.2mm_M3, F.Cu at (111.6, 72.3)
- added H2: MountingHole, MountingHole:MountingHole_3.2mm_M3, F.Cu at (111.6, 40.6)
- added H3: MountingHole, MountingHole:MountingHole_3.2mm_M3, F.Cu at (81.2, 64.7)
- added H3: MountingHole, MountingHole:MountingHole_3.2mm_M3, F.Cu at (81.2, 96.5)
- added H4: MountingHole, MountingHole:MountingHole_3.2mm_M3, F.Cu at (111.6, 64.7)
- added H4: MountingHole, MountingHole:MountingHole_3.2mm_M3, F.Cu at (111.6, 96.5)
- added J1: Conn_01x04_Socket, Connector_JST:JST_XH_B4B-XH-A_1x04_P2.50mm_Vertical, F.Cu at (81.6, 49.1)
- added J1: Conn_01x04_Socket, Connector_JST:JST_XH_B4B-XH-A_1x04_P2.50mm_Vertical, F.Cu at (81.6, 80.9)
- added LS1: Speaker_Ultrasound, uFinder:ULTRASONIC_16MM, B.Cu at (105.8, 52.7)
- added LS1: Speaker_Ultrasound, uFinder:ULTRASONIC_16MM, B.Cu at (105.8, 84.5)
- added Logo1: ~, uFinder:logo, B.Cu at (101.8, 40.2)
- added Logo1: ~, uFinder:logo, B.Cu at (101.8, 72.0)
- added Q1: MMBT3904, Package_TO_SOT_SMD:SOT-23, F.Cu at (86.4, 44.1)
- added Q1: MMBT3904, Package_TO_SOT_SMD:SOT-23, F.Cu at (86.4, 75.8)
- added Q2: MMBT3904, Package_TO_SOT_SMD:SOT-23, F.Cu at (87.3, 63.5)
- added Q2: MMBT3904, Package_TO_SOT_SMD:SOT-23, F.Cu at (87.3, 95.3)
- added R1: 10K, Resistor_SMD:R_0805_2012Metric, F.Cu at (107.7, 92.4)
- added R1: 10K, Resistor_SMD:R_0805_2012Metric, F.Cu at (107.7, 60.7)
- added R10: 10K, Resistor_SMD:R_0805_2012Metric, F.Cu at (89.2, 91.6)
- added R10: 10K, Resistor_SMD:R_0805_2012Metric, F.Cu at (89.2, 59.9)
- added R11: 1K, Resistor_SMD:R_0805_2012Metric, F.Cu at (96.3, 97.4)
- added R11: 1K, Resistor_SMD:R_0805_2012Metric, F.Cu at (96.3, 65.7)
- added R12: 3.9K, Resistor_SMD:R_0805_2012Metric, F.Cu at (86.1, 59.0)
- added R12: 3.9K, Resistor_SMD:R_0805_2012Metric, F.Cu at (86.1, 90.7)
- added R13: 10K, Resistor_SMD:R_0805_2012Metric, F.Cu at (98.7, 91.3)
- added R13: 10K, Resistor_SMD:R_0805_2012Metric, F.Cu at (98.7, 59.5)
- added R14: 10K, Resistor_SMD:R_0805_2012Metric, F.Cu at (102.1, 80.8)
- added R14: 10K, Resistor_SMD:R_0805_2012Metric, F.Cu at (102.1, 49.0)
- added R15: 120K, Resistor_SMD:R_0805_2012Metric, F.Cu at (90.8, 74.9)
- added R15: 120K, Resistor_SMD:R_0805_2012Metric, F.Cu at (90.8, 43.1)
- added R16: 2M, Resistor_SMD:R_0805_2012Metric, F.Cu at (90.6, 88.7)
- added R16: 2M, Resistor_SMD:R_0805_2012Metric, F.Cu at (90.6, 57.0)
- added R17: 10K, Resistor_SMD:R_0805_2012Metric, F.Cu at (85.7, 50.6)
- added R17: 10K, Resistor_SMD:R_0805_2012Metric, F.Cu at (85.7, 82.4)
- added R18: 100, Resistor_SMD:R_0805_2012Metric, F.Cu at (90.2, 95.0)
- added R18: 100, Resistor_SMD:R_0805_2012Metric, F.Cu at (90.2, 63.3)
- added R19: DO NOT POPULATE, Resistor_SMD:R_0805_2012Metric, F.Cu at (109.5, 58.1)
- added R19: DO NOT POPULATE, Resistor_SMD:R_0805_2012Metric, F.Cu at (109.5, 89.9)
- added R2: 75K, Resistor_SMD:R_0805_2012Metric, F.Cu at (102.0, 56.7)
- added R2: 75K, Resistor_SMD:R_0805_2012Metric, F.Cu at (102.0, 88.4)
- added R3: 6.8K, Resistor_SMD:R_0805_2012Metric, F.Cu at (107.4, 55.0)
- added R3: 6.8K, Resistor_SMD:R_0805_2012Metric, F.Cu at (107.4, 86.7)
- added R4: 220, Resistor_SMD:R_0805_2012Metric, F.Cu at (107.4, 84.7)
- added R4: 220, Resistor_SMD:R_0805_2012Metric, F.Cu at (107.4, 52.9)
- added R5: 75K, Resistor_SMD:R_0805_2012Metric, F.Cu at (109.0, 78.5)
- added R5: 75K, Resistor_SMD:R_0805_2012Metric, F.Cu at (109.0, 46.8)
- added R6: 10K, Resistor_SMD:R_0805_2012Metric, F.Cu at (99.8, 43.1)
- added R6: 10K, Resistor_SMD:R_0805_2012Metric, F.Cu at (99.8, 74.9)
- added R7: 75K, Resistor_SMD:R_0805_2012Metric, F.Cu at (93.7, 76.9)
- added R7: 75K, Resistor_SMD:R_0805_2012Metric, F.Cu at (93.7, 45.2)
- added R8: 4.3K, Resistor_SMD:R_0805_2012Metric, F.Cu at (90.6, 48.6)
- added R8: 4.3K, Resistor_SMD:R_0805_2012Metric, F.Cu at (90.6, 80.3)
- added R9: 120K, Resistor_SMD:R_0805_2012Metric, F.Cu at (95.2, 93.9)
- added R9: 120K, Resistor_SMD:R_0805_2012Metric, F.Cu at (95.2, 62.1)
- added TP1: TestPoint, uFinder:TestPoint_THTPad_D1.5mm_Drill0.7mm, B.Cu at (113.1, 59.7)
- added TP1: TestPoint, uFinder:TestPoint_THTPad_D1.5mm_Drill0.7mm, B.Cu at (113.1, 91.4)
- added TP2: TestPoint, uFinder:TestPoint_THTPad_D1.5mm_Drill0.7mm, B.Cu at (86.3, 39.2)
- added TP2: TestPoint, uFinder:TestPoint_THTPad_D1.5mm_Drill0.7mm, B.Cu at (86.3, 70.9)
- added TP3: TestPoint, uFinder:TestPoint_THTPad_D1.5mm_Drill0.7mm, B.Cu at (106.5, 42.8)
- added TP3: TestPoint, uFinder:TestPoint_THTPad_D1.5mm_Drill0.7mm, B.Cu at (106.5, 74.6)
- added TP4: TestPoint, uFinder:TestPoint_THTPad_D1.5mm_Drill0.7mm, B.Cu at (100.3, 95.2)
- added TP4: TestPoint, uFinder:TestPoint_THTPad_D1.5mm_Drill0.7mm, B.Cu at (100.3, 63.5)
- added TP5: TestPoint, uFinder:TestPoint_THTPad_D1.5mm_Drill0.7mm, B.Cu at (94.6, 72.8)
- added TP5: TestPoint, uFinder:TestPoint_THTPad_D1.5mm_Drill0.7mm, B.Cu at (94.6, 41.1)
- added TP6: TestPoint, uFinder:TestPoint_THTPad_D1.5mm_Drill0.7mm, B.Cu at (89.8, 45.9)
- added TP6: TestPoint, uFinder:TestPoint_THTPad_D1.5mm_Drill0.7mm, B.Cu at (89.8, 77.7)
- added TP7: TestPoint, uFinder:TestPoint_THTPad_D1.5mm_Drill0.7mm, B.Cu at (92.4, 91.6)
- added TP7: TestPoint, uFinder:TestPoint_THTPad_D1.5mm_Drill0.7mm, B.Cu at (92.4, 59.9)
- added TP8: TestPoint, uFinder:TestPoint_THTPad_D1.5mm_Drill0.7mm, B.Cu at (83.9, 92.5)
- added TP8: TestPoint, uFinder:TestPoint_THTPad_D1.5mm_Drill0.7mm, B.Cu at (83.9, 60.8)
- added U1: LM324, Package_SO:SOIC-14_3.9x8.7mm_P1.27mm, F.Cu at (96.2, 84.1)
- added U1: LM324, Package_SO:SOIC-14_3.9x8.7mm_P1.27mm, F.Cu at (96.2, 52.4)
Routing:
- net +3.3V: track 195.3 -> 102.0 mm, vias 8 -> 4
- net /DATA: track 210.2 -> 149.1 mm
- net Net-(U1A-+): track 66.4 -> 123.0 mm
- net Net-(D1-A): track 122.8 -> 79.5 mm
- net Net-(U1B--): track 74.0 -> 37.0 mm, vias 8 -> 4
- net (no net): track 0.00 -> 35.7 mm
- net Net-(U1B-+): track 147.6 -> 113.1 mm
- net Net-(Q1-C): track 151.1 -> 120.9 mm
- net Net-(Q3-B): track 37.9 -> 19.0 mm
- net Net-(U1C--): track 81.8 -> 64.9 mm
- net Net-(R7-Pad2): track 55.3 -> 39.6 mm, vias 8 -> 4
- net Net-(U1D--): track 72.2 -> 86.9 mm
- net GND: track 86.8 -> 72.2 mm
- net Net-(Q1-B): track 47.2 -> 33.2 mm
- net Net-(D1-K): track 31.7 -> 20.3 mm
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- added copper zone on F.Cu, net +3.3V
Other:
- board size 96.5 x 86.4 mm -> 96.5 x 100.3 mm
- board text added: "3.3V"

Commit message: updated panel
Parts:
- removed the C1 at (103.8, 60.7)
- removed the C1 at (103.8, 92.5)
- removed the C2 at (107.4, 50.8)
- removed the C2 at (107.4, 82.6)
- removed the C3 at (112.9, 78.5)
- removed the C3 at (112.9, 46.8)
- removed the C4 at (110.9, 78.4)
- removed the C4 at (110.9, 46.6)
- removed the C5 at (96.6, 44.2)
- removed the C5 at (96.6, 76.0)
- removed the C6 at (90.6, 52.4)
- removed the C6 at (90.6, 84.1)
- removed the C7 at (102.2, 51.2)
- removed the C7 at (102.2, 83.0)
- removed the C8 at (102.2, 85.4)
- removed the C8 at (102.2, 53.6)
- removed the C9 at (90.6, 54.9)
- removed the C9 at (90.6, 86.6)
- removed the D1 at (92.4, 63.3)
- removed the D1 at (92.4, 95.0)
- removed the H1 at (81.2, 40.6)
- removed the H1 at (81.2, 72.3)
- removed the H2 at (111.6, 72.3)
- removed the H2 at (111.6, 40.6)
- removed the H3 at (81.2, 64.7)
- removed the H3 at (81.2, 96.5)
- removed the H4 at (111.6, 64.7)
- removed the H4 at (111.6, 96.5)
- removed the J1 at (81.6, 49.1)
- removed the J1 at (81.6, 80.9)
- removed the LS1 at (105.8, 52.7)
- removed the LS1 at (105.8, 84.5)
- removed the Logo1 at (101.8, 40.2)
- removed the Logo1 at (101.8, 72.0)
- removed the Q1 at (86.4, 44.1)
- removed the Q1 at (86.4, 75.8)
- removed the Q2 at (87.3, 63.5)
- removed the Q2 at (87.3, 95.3)
- removed the R1 at (107.7, 92.4)
- removed the R1 at (107.7, 60.7)
- removed the R10 at (89.2, 91.6)
- removed the R10 at (89.2, 59.9)
- removed the R11 at (96.3, 97.4)
- removed the R11 at (96.3, 65.7)
- removed the R12 at (86.1, 59.0)
- removed the R12 at (86.1, 90.7)
- removed the R13 at (98.7, 91.3)
- removed the R13 at (98.7, 59.5)
- removed the R14 at (102.1, 80.8)
- removed the R14 at (102.1, 49.0)
- removed the R15 at (90.8, 74.9)
- removed the R15 at (90.8, 43.1)
- removed the R16 at (90.6, 88.7)
- removed the R16 at (90.6, 57.0)
- removed the R17 at (85.7, 50.6)
- removed the R17 at (85.7, 82.4)
- removed the R18 at (90.2, 95.0)
- removed the R18 at (90.2, 63.3)
- removed the R19 at (109.5, 58.1)
- removed the R19 at (109.5, 89.9)
- removed the R2 at (102.0, 56.7)
- removed the R2 at (102.0, 88.4)
- removed the R3 at (107.4, 55.0)
- removed the R3 at (107.4, 86.7)
- removed the R4 at (107.4, 84.7)
- removed the R4 at (107.4, 52.9)
- removed the R5 at (109.0, 78.5)
- removed the R5 at (109.0, 46.8)
- removed the R6 at (99.8, 43.1)
- removed the R6 at (99.8, 74.9)
- removed the R7 at (93.7, 76.9)
- removed the R7 at (93.7, 45.2)
- removed the R8 at (90.6, 48.6)
- removed the R8 at (90.6, 80.3)
- removed the R9 at (95.2, 93.9)
- removed the R9 at (95.2, 62.1)
- removed the TP1 at (113.1, 59.7)
- removed the TP1 at (113.1, 91.4)
- removed the TP2 at (86.3, 39.2)
- removed the TP2 at (86.3, 70.9)
- removed the TP3 at (106.5, 42.8)
- removed the TP3 at (106.5, 74.6)
- removed the TP4 at (100.3, 95.2)
- removed the TP4 at (100.3, 63.5)
- removed the TP5 at (94.6, 72.8)
- removed the TP5 at (94.6, 41.1)
- removed the TP6 at (89.8, 45.9)
- removed the TP6 at (89.8, 77.7)
- removed the TP7 at (92.4, 91.6)
- removed the TP7 at (92.4, 59.9)
- removed the TP8 at (83.9, 92.5)
- removed the TP8 at (83.9, 60.8)
- removed the U1 at (96.2, 84.1)
- removed the U1 at (96.2, 52.4)
- added C1: 10nF, Capacitor_SMD:C_0805_2012Metric, F.Cu at (89.2, 76.4)
- added C1: 10nF, Capacitor_SMD:C_0805_2012Metric, F.Cu at (89.2, 44.7)
- added C2: 1nF, Capacitor_SMD:C_0805_2012Metric, F.Cu at (85.6, 54.6)
- added C2: 1nF, Capacitor_SMD:C_0805_2012Metric, F.Cu at (85.6, 86.3)
- added C3: 1nF, Capacitor_SMD:C_0805_2012Metric, F.Cu at (80.0, 58.6)
- added C3: 1nF, Capacitor_SMD:C_0805_2012Metric, F.Cu at (80.0, 90.4)
- added C4: 68pF, Capacitor_SMD:C_0603_1608Metric, F.Cu at (82.0, 90.5)
- added C4: 68pF, Capacitor_SMD:C_0603_1608Metric, F.Cu at (82.0, 58.8)
- added C5: 10nF, Capacitor_SMD:C_0805_2012Metric, F.Cu at (96.3, 61.2)
- added C5: 10nF, Capacitor_SMD:C_0805_2012Metric, F.Cu at (96.3, 92.9)
- added C6: 1uF, Capacitor_SMD:C_0805_2012Metric, F.Cu at (102.3, 53.0)
- added C6: 1uF, Capacitor_SMD:C_0805_2012Metric, F.Cu at (102.3, 84.8)
- added C7: 1nF, Capacitor_SMD:C_0805_2012Metric, F.Cu at (90.8, 54.2)
- added C7: 1nF, Capacitor_SMD:C_0805_2012Metric, F.Cu at (90.8, 85.9)
- added C8: 1uF, Capacitor_SMD:C_0805_2012Metric, F.Cu at (90.8, 83.5)
- added C8: 1uF, Capacitor_SMD:C_0805_2012Metric, F.Cu at (90.8, 51.8)
- added C9: 1nF, Capacitor_SMD:C_0805_2012Metric, F.Cu at (102.3, 50.5)
- added C9: 1nF, Capacitor_SMD:C_0805_2012Metric, F.Cu at (102.3, 82.3)
- added D1: LED, LED_SMD:LED_0805_2012Metric, F.Cu at (100.5, 42.1)
- added D1: LED, LED_SMD:LED_0805_2012Metric, F.Cu at (100.5, 73.9)
- added H1: MountingHole, MountingHole:MountingHole_3.2mm_M3, F.Cu at (111.7, 64.8)
- added H1: MountingHole, MountingHole:MountingHole_3.2mm_M3, F.Cu at (111.7, 96.6)
- added H2: MountingHole, MountingHole:MountingHole_3.2mm_M3, F.Cu at (81.3, 96.6)
- added H2: MountingHole, MountingHole:MountingHole_3.2mm_M3, F.Cu at (81.3, 64.8)
- added H3: MountingHole, MountingHole:MountingHole_3.2mm_M3, F.Cu at (111.7, 40.7)
- added H3: MountingHole, MountingHole:MountingHole_3.2mm_M3, F.Cu at (111.7, 72.4)
- added H4: MountingHole, MountingHole:MountingHole_3.2mm_M3, F.Cu at (81.3, 40.7)
- added H4: MountingHole, MountingHole:MountingHole_3.2mm_M3, F.Cu at (81.3, 72.4)
- added J1: Conn_01x04_Socket, Connector_JST:JST_XH_B4B-XH-A_1x04_P2.50mm_Vertical, F.Cu at (111.4, 56.3)
- added J1: Conn_01x04_Socket, Connector_JST:JST_XH_B4B-XH-A_1x04_P2.50mm_Vertical, F.Cu at (111.4, 88.0)
- added LS1: Speaker_Ultrasound, uFinder:ULTRASONIC_16MM, B.Cu at (87.2, 84.4)
- added LS1: Speaker_Ultrasound, uFinder:ULTRASONIC_16MM, B.Cu at (87.2, 52.7)
- added Logo1: ~, uFinder:logo, B.Cu at (91.2, 65.2)
- added Logo1: ~, uFinder:logo, B.Cu at (91.2, 96.9)
- added Q1: MMBT3904, Package_TO_SOT_SMD:SOT-23, F.Cu at (106.6, 61.3)
- added Q1: MMBT3904, Package_TO_SOT_SMD:SOT-23, F.Cu at (106.6, 93.1)
- added Q2: MMBT3904, Package_TO_SOT_SMD:SOT-23, F.Cu at (105.7, 41.9)
- added Q2: MMBT3904, Package_TO_SOT_SMD:SOT-23, F.Cu at (105.7, 73.6)
- added R1: 10K, Resistor_SMD:R_0805_2012Metric, F.Cu at (85.2, 44.7)
- added R1: 10K, Resistor_SMD:R_0805_2012Metric, F.Cu at (85.2, 76.5)
- added R10: 10K, Resistor_SMD:R_0805_2012Metric, F.Cu at (103.8, 45.5)
- added R10: 10K, Resistor_SMD:R_0805_2012Metric, F.Cu at (103.8, 77.3)
- added R11: 1K, Resistor_SMD:R_0805_2012Metric, F.Cu at (96.7, 71.5)
- added R11: 1K, Resistor_SMD:R_0805_2012Metric, F.Cu at (96.7, 39.7)
- added R12: 3.9K, Resistor_SMD:R_0805_2012Metric, F.Cu at (106.8, 46.4)
- added R12: 3.9K, Resistor_SMD:R_0805_2012Metric, F.Cu at (106.8, 78.2)
- added R13: 10K, Resistor_SMD:R_0805_2012Metric, F.Cu at (94.3, 77.6)
- added R13: 10K, Resistor_SMD:R_0805_2012Metric, F.Cu at (94.3, 45.9)
- added R14: 10K, Resistor_SMD:R_0805_2012Metric, F.Cu at (90.8, 56.4)
- added R14: 10K, Resistor_SMD:R_0805_2012Metric, F.Cu at (90.8, 88.1)
- added R15: 120K, Resistor_SMD:R_0805_2012Metric, F.Cu at (102.2, 94.0)
- added R15: 120K, Resistor_SMD:R_0805_2012Metric, F.Cu at (102.2, 62.3)
- added R16: 2M, Resistor_SMD:R_0805_2012Metric, F.Cu at (102.3, 48.4)
- added R16: 2M, Resistor_SMD:R_0805_2012Metric, F.Cu at (102.3, 80.2)
- added R17: 10K, Resistor_SMD:R_0805_2012Metric, F.Cu at (107.3, 86.5)
- added R17: 10K, Resistor_SMD:R_0805_2012Metric, F.Cu at (107.3, 54.8)
- added R18: 100, Resistor_SMD:R_0805_2012Metric, F.Cu at (102.8, 73.9)
- added R18: 100, Resistor_SMD:R_0805_2012Metric, F.Cu at (102.8, 42.1)
- added R19: DO NOT POPULATE, Resistor_SMD:R_0805_2012Metric, F.Cu at (83.5, 79.0)
- added R19: DO NOT POPULATE, Resistor_SMD:R_0805_2012Metric, F.Cu at (83.5, 47.3)
- added R2: 75K, Resistor_SMD:R_0805_2012Metric, F.Cu at (91.0, 80.5)
- added R2: 75K, Resistor_SMD:R_0805_2012Metric, F.Cu at (91.0, 48.7)
- added R3: 6.8K, Resistor_SMD:R_0805_2012Metric, F.Cu at (85.6, 50.4)
- added R3: 6.8K, Resistor_SMD:R_0805_2012Metric, F.Cu at (85.6, 82.2)
- added R4: 220, Resistor_SMD:R_0805_2012Metric, F.Cu at (85.6, 84.2)
- added R4: 220, Resistor_SMD:R_0805_2012Metric, F.Cu at (85.6, 52.5)
- added R5: 75K, Resistor_SMD:R_0805_2012Metric, F.Cu at (84.0, 90.4)
- added R5: 75K, Resistor_SMD:R_0805_2012Metric, F.Cu at (84.0, 58.6)
- added R6: 10K, Resistor_SMD:R_0805_2012Metric, F.Cu at (93.2, 62.3)
- added R6: 10K, Resistor_SMD:R_0805_2012Metric, F.Cu at (93.2, 94.0)
- added R7: 75K, Resistor_SMD:R_0805_2012Metric, F.Cu at (99.2, 92.0)
- added R7: 75K, Resistor_SMD:R_0805_2012Metric, F.Cu at (99.2, 60.2)
- added R8: 4.3K, Resistor_SMD:R_0805_2012Metric, F.Cu at (102.3, 88.6)
- added R8: 4.3K, Resistor_SMD:R_0805_2012Metric, F.Cu at (102.3, 56.8)
- added R9: 120K, Resistor_SMD:R_0805_2012Metric, F.Cu at (97.8, 43.3)
- added R9: 120K, Resistor_SMD:R_0805_2012Metric, F.Cu at (97.8, 75.0)
- added TP1: TestPoint, uFinder:TestPoint_THTPad_D1.5mm_Drill0.7mm, B.Cu at (79.9, 77.5)
- added TP1: TestPoint, uFinder:TestPoint_THTPad_D1.5mm_Drill0.7mm, B.Cu at (79.9, 45.7)
- added TP2: TestPoint, uFinder:TestPoint_THTPad_D1.5mm_Drill0.7mm, B.Cu at (106.7, 98.0)
- added TP2: TestPoint, uFinder:TestPoint_THTPad_D1.5mm_Drill0.7mm, B.Cu at (106.7, 66.2)
- added TP3: TestPoint, uFinder:TestPoint_THTPad_D1.5mm_Drill0.7mm, B.Cu at (86.5, 62.6)
- added TP3: TestPoint, uFinder:TestPoint_THTPad_D1.5mm_Drill0.7mm, B.Cu at (86.5, 94.3)
- added TP4: TestPoint, uFinder:TestPoint_THTPad_D1.5mm_Drill0.7mm, B.Cu at (92.7, 41.9)
- added TP4: TestPoint, uFinder:TestPoint_THTPad_D1.5mm_Drill0.7mm, B.Cu at (92.7, 73.7)
- added TP5: TestPoint, uFinder:TestPoint_THTPad_D1.5mm_Drill0.7mm, B.Cu at (98.3, 96.1)
- added TP5: TestPoint, uFinder:TestPoint_THTPad_D1.5mm_Drill0.7mm, B.Cu at (98.3, 64.3)
- added TP6: TestPoint, uFinder:TestPoint_THTPad_D1.5mm_Drill0.7mm, B.Cu at (103.2, 59.5)
- added TP6: TestPoint, uFinder:TestPoint_THTPad_D1.5mm_Drill0.7mm, B.Cu at (103.2, 91.2)
- added TP7: TestPoint, uFinder:TestPoint_THTPad_D1.5mm_Drill0.7mm, B.Cu at (100.6, 77.3)
- added TP7: TestPoint, uFinder:TestPoint_THTPad_D1.5mm_Drill0.7mm, B.Cu at (100.6, 45.5)
- added TP8: TestPoint, uFinder:TestPoint_THTPad_D1.5mm_Drill0.7mm, B.Cu at (109.0, 76.4)
- added TP8: TestPoint, uFinder:TestPoint_THTPad_D1.5mm_Drill0.7mm, B.Cu at (109.0, 44.6)
- added U1: LM324, Package_SO:SOIC-14_3.9x8.7mm_P1.27mm, F.Cu at (96.8, 53.0)
- added U1: LM324, Package_SO:SOIC-14_3.9x8.7mm_P1.27mm, F.Cu at (96.8, 84.8)
